File: ODAmain/ODAmain/ODAmain.kicad_sch (KiCad schematic)
At the start: 53 parts, among them J1 EMC, J10 gh:CAN_2, J2 Conn_02x06_Counter_Clockwise, J3 Terminate_CAN1, J4 Conn_02x05_Counter_Clockwise, J4 Terminate_CAN2, J6 CAN_1, J7 CAN_2, J8 ENCODER1, J8 gh:ENCODER1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

Commit message: 2024/08/23
Other:
- removed sheet F446RE
- added sheet f446 (untitled.kicad_sch)
Changed lines of the file:
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@@
     (instances
       (project "ODAmain"
-        (path "/83972afe-ad2d-4cb7-a6d7-9dc26d3c5939/b550f57f-bdcc-4169-bf19-85d84ec7f50a"
-          (reference "J8") (unit 1)
-        )
         (path "/83972afe-ad2d-4cb7-a6d7-9dc26d3c5939"
           (reference "J8") (unit 1)
@@
     (instances
       (project "ODAmain"
-        (path "/83972afe-ad2d-4cb7-a6d7-9dc26d3c5939/b550f57f-bdcc-4169-bf19-85d84ec7f50a"
-          (reference "#PWR033") (unit 1)
-        )
         (path "/83972afe-ad2d-4cb7-a6d7-9dc26d3c5939"
           (reference "#PWR011") (unit 1)
@@
     (instances
       (project "ODAmain"
-        (path "/83972afe-ad2d-4cb7-a6d7-9dc26d3c5939/b550f57f-bdcc-4169-bf19-85d84ec7f50a"
-          (reference "J8") (unit 1)
-        )
         (path "/83972afe-ad2d-4cb7-a6d7-9dc26d3c5939"
           (reference "J11") (unit 1)
@@
     (instances
       (project "ODAmain"
-        (path "/83972afe-ad2d-4cb7-a6d7-9dc26d3c5939/b550f57f-bdcc-4169-bf19-85d84ec7f50a"
-          (reference "#PWR032") (unit 1)
-        )
         (path "/83972afe-ad2d-4cb7-a6d7-9dc26d3c5939"
           (reference "#PWR010") (unit 1)
@@
     )
   )
-  (sheet (at 20.32 162.56) (size 27.94 21.59) (fields_autoplaced)
-    (stroke (width 0) (type solid))
+  (sheet (at 31.75 167.64) (size 22.86 13.97) (fields_autoplaced)
+    (stroke (width 0.1524) (type solid))
     (fill (color 0 0 0 0.0000))
-    (property "Sheetname" "F446RE" (at 20.32 161.8484 0)
+    (property "Sheetname" "f446" (at 31.75 166.9284 0)
       (effects (font (size 1.27 1.27)) (justify left bottom))
     )
-    (property "Sheetfile" "F446RE.sch" (at 20.32 184.7346 0)
+    (property "Sheetfile" "untitled.kicad_sch" (at 31.75 182.1946 0)
       (effects (font (size 1.27 1.27)) (justify left top))
     )
