File: ODAmain/CAN_hab/CAN_hab.kicad_pcb (KiCad board)
At the start: 2 copper layers, 50 x 25 mm, 23 parts, among them J1 Terminate, J11 gh*2_4, J13 gh*2_5, J15 gh*2_6, J19 Terminate, J2 xh, J20 XT30, J21 XT30, J22 XT30, J4 gh*4_1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

Commit message: 2024/08/23
Parts:
- J20, J21, J22: footprint Connector_AMASS:AMASS_XT30UPB-M_1x02_P5.0mm_Vertical -> Connector_AMASS:AMASS_XT30U-F_1x02_P5.0mm_Vertical
Changed lines of the file:
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@@
   (net 7 "GNDPWR")
   (net 8 "Net-(J19-Pin_1)")
-  (footprint "Connector_AMASS:AMASS_XT30UPB-M_1x02_P5.0mm_Vertical" (layer "F.Cu")
+  (footprint "Connector_AMASS:AMASS_XT30U-F_1x02_P5.0mm_Vertical" (layer "F.Cu")
     (at 164.848 109.439)
-    (descr "Connector XT30 Vertical PCB Male, https://www.tme.eu/en/Document/4acc913878197f8c2e30d4b8cdc47230/XT30UPB%20SPEC.pdf")
+    (descr "Connector XT30 Vertical Cable Female, https://www.tme.eu/en/Document/3cbfa5cfa544d79584972dd5234a409e/XT30U%20SPEC.pdf")
     (tags "RC Connector XT30")
     (property "Sheetfile" "CAN_hab.kicad_sch")
@@
     (property "ki_keywords" "connector")
     (attr through_hole)
-    (fp_text reference "J22" (at 2.5 -3.32) (layer "F.Fab")
+    (fp_text reference "J22" (at 2.5 -4) (layer "F.SilkS")
         (effects (font (size 1 1) (thickness 0.15)))
     )
@@
         (effects (font (size 1 1) (thickness 0.15)))
     )
-    (fp_text user "+" (at 8.636 -0.272) (layer "F.SilkS")
+    (fp_text user "-" (at -4 0) (layer "F.SilkS")
+        (effects (font (size 1.5 1.5) (thickness 0.15)))
+    )
+    (fp_text user "+" (at 9 0) (layer "F.SilkS")
         (effects (font (size 1.5 1.5) (thickness 0.15)))
     )
@@
     (fp_line (start 7.6 -2.6) (end 7.6 2.6)
       (stroke (width 0.1) (type solid)) (layer "F.Fab"))
-    (pad "1" thru_hole rect (at 0 0) (size 3 3) (drill 1.8) (layers "*.Cu" "*.Mask")
+    (pad "1" thru_hole rect (at 0 0) (size 3.8 3.8) (drill 2.7) (layers "*.Cu" "*.Mask")
       (net 7 "GNDPWR") (pinfunction "Pin_1") (pintype "passive"))
-    (pad "2" thru_hole circle (at 5 0) (size 3 3) (drill 1.8) (layers "*.Cu" "*.Mask")
+    (pad "2" thru_hole circle (at 5 0) (size 4 4) (drill 2.7) (layers "*.Cu" "*.Mask")
       (net 6 "+BATT") (pinfunction "Pin_2") (pintype "passive"))
-    (model "${KICAD6_3DMODEL_DIR}/Connector_AMASS.3dshapes/AMASS_XT30UPB-M_1x02_P5.0mm_Vertical.wrl"
+    (model "${KICAD6_3DMODEL_DIR}/Connector_AMASS.3dshapes/AMASS_XT30U-F_1x02_P5.0mm_Vertical.wrl"
       (offset (xyz 0 0 0))
       (scale (xyz 1 1 1))
@@
     )
   )
-  (footprint "Connector_AMASS:AMASS_XT30UPB-M_1x02_P5.0mm_Vertical" (layer "F.Cu")
+  (footprint "Connector_AMASS:AMASS_XT30U-F_1x02_P5.0mm_Vertical" (layer "F.Cu")
     (at 152.148 109.439)
-    (descr "Connector XT30 Vertical PCB Male, https://www.tme.eu/en/Document/4acc913878197f8c2e30d4b8cdc47230/XT30UPB%20SPEC.pdf")
+    (descr "Connector XT30 Vertical Cable Female, https://www.tme.eu/en/Document/3cbfa5cfa544d79584972dd5234a409e/XT30U%20SPEC.pdf")
     (tags "RC Connector XT30")
     (property "Sheetfile" "CAN_hab.kicad_sch")
@@
     (property "ki_keywords" "connector")
     (attr through_hole)
-    (fp_text reference "J21" (at 2.54 -3.32) (layer "F.Fab")
+    (fp_text reference "J21" (at 2.5 -4) (layer "F.SilkS")
         (effects (font (size 1 1) (thickness 0.15)))
     )
@@
         (effects (font (size 1 1) (thickness 0.15)))
     )
-    (fp_text user "+" (at 8.76 -0.272) (layer "F.SilkS")
+    (fp_text user "+" (at 9 0) (layer "F.SilkS")
+        (effects (font (size 1.5 1.5) (thickness 0.15)))
+    )
+    (fp_text user "-" (at -4 0) (layer "F.SilkS")
         (effects (font (size 1.5 1.5) (thickness 0.15)))
     )
@@
     (fp_line (start 7.6 -2.6) (end 7.6 2.6)
       (stroke (width 0.1) (type solid)) (layer "F.Fab"))
-    (pad "1" thru_hole rect (at 0 0) (size 3 3) (drill 1.8) (layers "*.Cu" "*.Mask")
+    (pad "1" thru_hole rect (at 0 0) (size 3.8 3.8) (drill 2.7) (layers "*.Cu" "*.Mask")
       (net 7 "GNDPWR") (pinfunction "Pin_1") (pintype "passive"))
-    (pad "2" thru_hole circle (at 5 0) (size 3 3) (drill 1.8) (layers "*.Cu" "*.Mask")
+    (pad "2" thru_hole circle (at 5 0) (size 4 4) (drill 2.7) (layers "*.Cu" "*.Mask")
       (net 6 "+BATT") (pinfunction "Pin_2") (pintype "passive"))
-    (model "${KICAD6_3DMODEL_DIR}/Connector_AMASS.3dshapes/AMASS_XT30UPB-M_1x02_P5.0mm_Vertical.wrl"
+    (model "${KICAD6_3DMODEL_DIR}/Connector_AMASS.3dshapes/AMASS_XT30U-F_1x02_P5.0mm_Vertical.wrl"
       (offset (xyz 0 0 0))
       (scale (xyz 1 1 1))
@@
     (pad "~" thru_hole circle (at 2.2 0) (size 1 1) (drill 0.3) (layers "*.Cu" "*.Mask"))
   )
-  (footprint "Connector_AMASS:AMASS_XT30UPB-M_1x02_P5.0mm_Vertical" (layer "F.Cu")
+  (footprint "Connector_AMASS:AMASS_XT30U-F_1x02_P5.0mm_Vertical" (layer "F.Cu")
     (at 139.528 109.439)
-    (descr "Connector XT30 Vertical PCB Male, https://www.tme.eu/en/Document/4acc913878197f8c2e30d4b8cdc47230/XT30UPB%20SPEC.pdf")
+    (descr "Connector XT30 Vertical Cable Female, https://www.tme.eu/en/Document/3cbfa5cfa544d79584972dd5234a409e/XT30U%20SPEC.pdf")
     (tags "RC Connector XT30")
     (property "Sheetfile" "CAN_hab.kicad_sch")
@@
     (property "ki_keywords" "connector")
     (attr through_hole)
-    (fp_text reference "J20" (at 2.46 -3.32) (layer "F.Fab")
+    (fp_text reference "J20" (at 2.5 -4) (layer "F.SilkS")
         (effects (font (size 1 1) (thickness 0.15)))
     )
@@
         (effects (font (size 1 1) (thickness 0.15)))
     )
-    (fp_text user "+" (at 8.68 -0.272) (layer "F.SilkS")
+    (fp_text user "-" (at -4 0) (layer "F.SilkS")
+        (effects (font (size 1.5 1.5) (thickness 0.15)))
+    )
+    (fp_text user "+" (at 9 0) (layer "F.SilkS")
         (effects (font (size 1.5 1.5) (thickness 0.15)))
     )
@@
     (fp_line (start 7.6 -2.6) (end 7.6 2.6)
       (stroke (width 0.1) (type solid)) (layer "F.Fab"))
-    (pad "1" thru_hole rect (at 0 0) (size 3 3) (drill 1.8) (layers "*.Cu" "*.Mask")
+    (pad "1" thru_hole rect (at 0 0) (size 3.8 3.8) (drill 2.7) (layers "*.Cu" "*.Mask")
       (net 7 "GNDPWR") (pinfunction "Pin_1") (pintype "passive"))
-    (pad "2" thru_hole circle (at 5 0) (size 3 3) (drill 1.8) (layers "*.Cu" "*.Mask")
+    (pad "2" thru_hole circle (at 5 0) (size 4 4) (drill 2.7) (layers "*.Cu" "*.Mask")
       (net 6 "+BATT") (pinfunction "Pin_2") (pintype "passive"))
-    (model "${KICAD6_3DMODEL_DIR}/Connector_AMASS.3dshapes/AMASS_XT30UPB-M_1x02_P5.0mm_Vertical.wrl"
+    (model "${KICAD6_3DMODEL_DIR}/Connector_AMASS.3dshapes/AMASS_XT30U-F_1x02_P5.0mm_Vertical.wrl"
       (offset (xyz 0 0 0))
       (scale (xyz 1 1 1))
@@
         (xy 180.34 112.522)
         (xy 180.467 93.091)
-        (xy 180.467 93.091)
         (xy 173.863 93.091)
         (xy 173.863 104.14)
@@
         (xy 180.34 112.522)
         (xy 180.467 93.091)
-        (xy 180.467 93.091)
         (xy 173.863 93.091)

Commit message: 2024/09/22
Parts:
- added D1: CAN_H, Footprint_nishi:LED_0603_1608, F.Cu at (145.5, 96.0)
- added D2: CAN_L, Footprint_nishi:LED_0603_1608, F.Cu at (150.0, 96.0)
- added G***: LOGO, watanabe_smy:sabamiso_10^10, B.Cu at (140.1, 91.0)
- added R2: 1.5k, Footprint_nishi:R_0603_1608, B.Cu at (145.4, 96.0)
- added R3: 1.5k, Footprint_nishi:R_0603_1608, B.Cu at (149.9, 96.0)
- moved J20 6.15 mm to (145.7, 109.4), turned to 180 degrees
- moved J21 6.15 mm to (158.3, 109.4), turned to 180 degrees
- moved J22 6.15 mm to (171.0, 109.4), turned to 180 degrees
- moved G*** 1.73 mm to (167.0, 98.5)
Routing:
- net GND: track 0.00 -> 2.76 mm, vias 3 -> 5
- net CAN_L: track 92.7 -> 94.3 mm
- net CAN_H: track 93.3 -> 94.8 mm, vias 0 -> 1
- net Net-(D2-A): vias 0 -> 1
- net Net-(D1-A): vias 0 -> 1
Other:
- board text added: "September.05. 2024 @nnct_robo CANhab_ver2.0"
- board text removed: "April. 29. 2024 @nnct_robo CANhab"
