File: ODAmain/CAN_hab/CAN_hab.kicad_sch (KiCad schematic)
At the start: 18 parts, among them J1 Terminate, J11 gh*2_4, J13 gh*2_5, J15 gh*2_6, J19 Terminate, J2 xh, J4 gh*4_1, J5 gh*2_1, J6 gh*4_2, J7 XT30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

Commit message: 2024/09/22
Parts:
- added D1: CAN_H, Footprint_nishi:LED_0603_1608, symbol Device:LED
- added D2: CAN_L, Footprint_nishi:LED_0603_1608, symbol Device:LED
- added R2, R3: 1.5k, Footprint_nishi:R_0603_1608, symbol Device:R
- J7, J8, J9: footprint Connector_AMASS:AMASS_XT30UPB-M_1x02_P5.0mm_Vertical -> Connector_AMASS:AMASS_XT30U-F_1x02_P5.0mm_Vertical
Connections:
- net CAN_H: now also R2.1
- net CAN_L: now also R3.1
- net GND: now also D1.1 (K), D2.1 (K)
- new net: D2.2 (A), R3.2
- new net: D1.2 (A), R2.2
Changed lines of the file:
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@@
+    )
+  )
+  (global_label "CAN_L" (shape input) (at 107.95 67.31 90) (fields_autoplaced)
+    (effects (font (size 1.27 1.27)) (justify left))
+    (property "Intersheetrefs" "${INTERSHEET_REFS}" (at 107.95 58.64 90)
+      (effects (font (size 1.27 1.27)) (justify left) hide)
     )
   )
@@
     )
   )
+  (global_label "CAN_H" (shape input) (at 100.33 67.31 90) (fields_autoplaced)
+    (effects (font (size 1.27 1.27)) (justify left))
+    (property "Intersheetrefs" "${INTERSHEET_REFS}" (at 100.33 58.3376 90)
+      (effects (font (size 1.27 1.27)) (justify left) hide)
+    )
+  )
   (symbol (lib_id "Connector_Generic:Conn_01x02") (at 238.76 83.82 180) (unit 1)
     (in_bom yes) (on_board yes) (dnp no)
@@
     )
   )
+  (symbol (lib_id "Device:R") (at 107.95 71.12 0) (unit 1)
+    (in_bom yes) (on_board yes) (dnp no) (fields_autoplaced)
+    (property "Reference" "R3" (at 110.49 69.85 0)
+      (effects (font (size 1.27 1.27)) (justify left))
+    )
+    (property "Value" "1.5k" (at 110.49 72.39 0)
+      (effects (font (size 1.27 1.27)) (justify left))
+    )
+    (property "Footprint" "Footprint_nishi:R_0603_1608" (at 106.172 71.12 90)
+      (effects (font (size 1.27 1.27)) hide)
+    )
+    (property "Datasheet" "~" (at 107.95 71.12 0)
+      (effects (font (size 1.27 1.27)) hide)
+    )
+    (pin "1")
+    (pin "2")
+    (instances
+      (project "CAN_hab"
+        (path "/b09c36ba-556c-4362-b936-bc1f1ef98ff1"
+          (reference "R3") (unit 1)
+        )
+      )
+    )
+  )
+  (symbol (lib_id "power:GND") (at 107.95 82.55 0) (unit 1)
+    (in_bom yes) (on_board yes) (dnp no) (fields_autoplaced)
+    (property "Reference" "#PWR06" (at 107.95 88.9 0)
+      (effects (font (size 1.27 1.27)) hide)
+    )
+    (property "Value" "GND" (at 107.95 87.63 0)
+      (effects (font (size 1.27 1.27)))
+    )
+    (property "Footprint" "" (at 107.95 82.55 0)
+      (effects (font (size 1.27 1.27)) hide)
+    )
+    (property "Datasheet" "" (at 107.95 82.55 0)
+      (effects (font (size 1.27 1.27)) hide)
+    )
+    (pin "1")
+    (instances
+      (project "CAN_hab"
+        (path "/b09c36ba-556c-4362-b936-bc1f1ef98ff1"
+          (reference "#PWR06") (unit 1)
+        )
+      )
+    )
+  )
   (symbol (lib_id "Connector_Generic:Conn_01x02") (at 200.66 83.82 180) (unit 1)
     (in_bom yes) (on_board yes) (dnp no)
@@
       (effects (font (size 1.27 1.27)) (justify left))
     )
-    (property "Footprint" "Connector_AMASS:AMASS_XT30UPB-M_1x02_P5.0mm_Vertical" (at 200.66 83.82 0)
+    (property "Footprint" "Connector_AMASS:AMASS_XT30U-F_1x02_P5.0mm_Vertical" (at 200.66 83.82 0)
       (effects (font (size 1.27 1.27)) hide)
     )
@@
     )
   )
+  (symbol (lib_id "Device:R") (at 100.33 71.12 0) (unit 1)
+    (in_bom yes) (on_board yes) (dnp no) (fields_autoplaced)
+    (property "Reference" "R2" (at 102.87 69.85 0)
+      (effects (font (size 1.27 1.27)) (justify left))
+    )
+    (property "Value" "1.5k" (at 102.87 72.39 0)
+      (effects (font (size 1.27 1.27)) (justify left))
+    )
+    (property "Footprint" "Footprint_nishi:R_0603_1608" (at 98.552 71.12 90)
+      (effects (font (size 1.27 1.27)) hide)
+    )
+    (property "Datasheet" "~" (at 100.33 71.12 0)
+      (effects (font (size 1.27 1.27)) hide)
+    )
+    (pin "1")
+    (pin "2")
+    (instances
+      (project "CAN_hab"
+        (path "/b09c36ba-556c-4362-b936-bc1f1ef98ff1"
+          (reference "R2") (unit 1)
+        )
+      )
+    )
+  )
+  (symbol (lib_id "Device:LED") (at 107.95 78.74 90) (unit 1)
+    (in_bom yes) (on_board yes) (dnp no) (fields_autoplaced)
+    (property "Reference" "D2" (at 111.76 79.0575 90)
+      (effects (font (size 1.27 1.27)) (justify right))
+    )
+    (property "Value" "CAN_L" (at 111.76 81.5975 90)
+      (effects (font (size 1.27 1.27)) (justify right))
+    )
+    (property "Footprint" "Footprint_nishi:LED_0603_1608" (at 107.95 78.74 0)
+      (effects (font (size 1.27 1.27)) hide)
+    )
+    (property "Datasheet" "~" (at 107.95 78.74 0)
+      (effects (font (size 1.27 1.27)) hide)
+    )
+    (pin "1")
+    (pin "2")
+    (instances
+      (project "CAN_hab"
+        (path "/b09c36ba-556c-4362-b936-bc1f1ef98ff1"
+          (reference "D2") (unit 1)
+        )
+      )
+    )
+  )
   (symbol (lib_id "Connector_Generic:Conn_01x04") (at 49.53 78.74 0) (unit 1)
     (in_bom yes) (on_board yes) (dnp no) (fields_autoplaced)
@@
     )
   )
+  (symbol (lib_id "power:GND") (at 100.33 82.55 0) (unit 1)
+    (in_bom yes) (on_board yes) (dnp no) (fields_autoplaced)
+    (property "Reference" "#PWR05" (at 100.33 88.9 0)
+      (effects (font (size 1.27 1.27)) hide)
+    )
+    (property "Value" "GND" (at 100.33 87.63 0)
+      (effects (font (size 1.27 1.27)))
+    )
+    (property "Footprint" "" (at 100.33 82.55 0)
+      (effects (font (size 1.27 1.27)) hide)
+    )
+    (property "Datasheet" "" (at 100.33 82.55 0)
+      (effects (font (size 1.27 1.27)) hide)
+    )
+    (pin "1")
+    (instances
+      (project "CAN_hab"
+        (path "/b09c36ba-556c-4362-b936-bc1f1ef98ff1"
+          (reference "#PWR05") (unit 1)
+        )
+      )
+    )
+  )
   (symbol (lib_id "power:GNDPWR") (at 243.84 83.82 0) (mirror y) (unit 1)
     (in_bom yes) (on_board yes) (dnp no)
@@
       (effects (font (size 1.27 1.27)) (justify left))
     )
-    (property "Footprint" "Connector_AMASS:AMASS_XT30UPB-M_1x02_P5.0mm_Vertical" (at 213.36 83.82 0)
+    (property "Footprint" "Connector_AMASS:AMASS_XT30U-F_1x02_P5.0mm_Vertical" (at 213.36 83.82 0)
       (effects (font (size 1.27 1.27)) hide)
     )
@@
       (effects (font (size 1.27 1.27)) (justify left))
     )
-    (property "Footprint" "Connector_AMASS:AMASS_XT30UPB-M_1x02_P5.0mm_Vertical" (at 226.06 83.82 0)
+    (property "Footprint" "Connector_AMASS:AMASS_XT30U-F_1x02_P5.0mm_Vertical" (at 226.06 83.82 0)
       (effects (font (size 1.27 1.27)) hide)
     )
@@
         )
       )
+    )
+  )
+  (symbol (lib_id "Device:LED") (at 100.33 78.74 90) (unit 1)
+    (in_bom yes) (on_board yes) (dnp no) (fields_autoplaced)
+    (property "Reference" "D1" (at 104.14 79.0575 90)
+      (effects (font (size 1.27 1.27)) (justify right))
+    )
+    (property "Value" "CAN_H" (at 104.14 81.5975 90)
+      (effects (font (size 1.27 1.27)) (justify right))
+    )
+    (property "Footprint" "Footprint_nishi:LED_0603_1608" (at 100.33 78.74 0)
+      (effects (font (size 1.27 1.27)) hide)
+    )
+    (property "Datasheet" "~" (at 100.33 78.74 0)
+      (effects (font (size 1.27 1.27)) hide)
+    )
+    (pin "1")
+    (pin "2")
+    (instances
+      (project "CAN_hab"
+        (path "/b09c36ba-556c-4362-b936-bc1f1ef98ff1"
+          (reference "D1") (unit 1)
+        )
+      )
