File: YAMADAmain_correct/YAMADAmain_correct.kicad_pcb (KiCad board)
At the start: 2 copper layers, 50 x 50 mm, 60 parts, among them J1 BATT, J2 Conn_02x06_Counter_Clockwise, J3 emc-sw, J4 Conn_02x05_Counter_Clockwise, J5 motor1, J6 motor2, J7 motor3, J8 motor4, U1 NJM2845DL1-33, U10 SW_DP3T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

Commit message: 2024/09/22
Parts:
- added IC1: BD7LS04G-CTL, BD7LS04G-CTL:SOT95P280X125-5N, B.Cu at (146.8, 106.8)
Changed lines of the file:
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@@
+    )
+  )
+  (footprint "BD7LS04G-CTL:SOT95P280X125-5N" (layer "B.Cu")
+    (at 146.8 106.85 -90)
+    (descr "SSOP5")
+    (tags "Integrated Circuit")
+    (property "Corestaff Part Number" "")
+    (property "Corestaff Price/Stock" "")
+    (property "Height" "1.25")
+    (property "Manufacturer_Name" "ROHM Semiconductor")
+    (property "Manufacturer_Part_Number" "BD7LS04G-CTL")
+    (property "Sheetfile" "YAMADAmain_ver2.0.kicad_sch")
+    (property "Sheetname" "")
+    (property "ki_description" "General Purpose CMOS Logic IC, Automotive Single Inverter, SSOP5")
+    (attr smd)
+    (fp_text reference "IC1" (at 0 0 90) (layer "B.Fab")
+        (effects (font (size 1.27 1.27) (thickness 0.254)) (justify mirror))
+    )
+    (fp_text value "BD7LS04G-CTL" (at 0 0 90) (layer "B.SilkS") hide
+        (effects (font (size 1.27 1.27) (thickness 0.254)) (justify mirror))
+    )
+    (fp_text user "${REFERENCE}" (at 0 0 90) (layer "B.Fab")
+        (effects (font (size 1.27 1.27) (thickness 0.254)) (justify mirror))
+    )
+    (fp_line (start -1.85 1.5) (end -0.95 1.5)
+      (stroke (width 0.2) (type solid)) (layer "B.SilkS"))
+    (fp_line (start -0.6 -1.45) (end -0.6 1.45)
+      (stroke (width 0.2) (type solid)) (layer "B.SilkS"))
+    (fp_line (start -0.6 1.45) (end 0.6 1.45)
+      (stroke (width 0.2) (type solid)) (layer "B.SilkS"))
+    (fp_line (start 0.6 -1.45) (end -0.6 -1.45)
+      (stroke (width 0.2) (type solid)) (layer "B.SilkS"))
+    (fp_line (start 0.6 1.45) (end 0.6 -1.45)
+      (stroke (width 0.2) (type solid)) (layer "B.SilkS"))
+    (fp_line (start -2.1 -1.8) (end -2.1 1.8)
+      (stroke (width 0.05) (type solid)) (layer "B.CrtYd"))
+    (fp_line (start -2.1 1.8) (end 2.1 1.8)
+      (stroke (width 0.05) (type solid)) (layer "B.CrtYd"))
+    (fp_line (start 2.1 -1.8) (end -2.1 -1.8)
+      (stroke (width 0.05) (type solid)) (layer "B.CrtYd"))
+    (fp_line (start 2.1 1.8) (end 2.1 -1.8)
+      (stroke (width 0.05) (type solid)) (layer "B.CrtYd"))
+    (fp_line (start -0.825 -1.45) (end -0.825 1.45)
+      (stroke (width 0.1) (type solid)) (layer "B.Fab"))
+    (fp_line (start -0.825 0.5) (end 0.125 1.45)
+      (stroke (width 0.1) (type solid)) (layer "B.Fab"))
+    (fp_line (start -0.825 1.45) (end 0.825 1.45)
+      (stroke (width 0.1) (type solid)) (layer "B.Fab"))
+    (fp_line (start 0.825 -1.45) (end -0.825 -1.45)
+      (stroke (width 0.1) (type solid)) (layer "B.Fab"))
+    (fp_line (start 0.825 1.45) (end 0.825 -1.45)
+      (stroke (width 0.1) (type solid)) (layer "B.Fab"))
+    (pad "1" smd rect (at -1.4 0.95 180) (size 0.6 0.9) (layers "B.Cu" "B.Paste" "B.Mask")
+      (pinfunction "N.C.") (pintype "no_connect"))
+    (pad "2" smd rect (at -1.4 0 180) (size 0.6 0.9) (layers "B.Cu" "B.Paste" "B.Mask")
+      (pinfunction "A") (pintype "passive"))
+    (pad "3" smd rect (at -1.4 -0.95 180) (size 0.6 0.9) (layers "B.Cu" "B.Paste" "B.Mask")
+      (pinfunction "GND") (pintype "passive"))
+    (pad "4" smd rect (at 1.4 -0.95 180) (size 0.6 0.9) (layers "B.Cu" "B.Paste" "B.Mask")
+      (pinfunction "Y") (pintype "passive"))
+    (pad "5" smd rect (at 1.4 0.95 180) (size 0.6 0.9) (layers "B.Cu" "B.Paste" "B.Mask")
+      (pinfunction "VCC") (pintype "passive"))
+    (model "BD7LS04G-CTL.stp"
+      (offset (xyz 0 0 0))
+      (scale (xyz 1 1 1))
+      (rotate (xyz 0 0 0))
     )
   )
