File: YAMADAmain_ver2.0/YAMADAmain_ver2.0.kicad_pcb (KiCad board)
At the start: 2 copper layers, 50 x 50 mm, 77 parts, among them IC1 BD7LS04G-CTL, J1 im920sl_USB, J10 RX==RX, J11 TX==TX, J2 BATT, J3 emc-sw_1, J4 motor1, J5 motor2, J6 motor3, J7 motor4, J8 RX==TX, J9 TX==RX, Q1 2SC3265-Y, U1 NJM2845DL1-33, U11 4.7k, U12 SW_DP3T, U13 0.1u, U14 0.1u, U15 D_Schottky, U16 4.7u, U17 ST-LINK, U18 STM32F446RETx-stm32, U19 0.1u, U2 IM920sL, U20 0.1u, U21 0.1u, U22 0.1u, U23 0.1u, U3 FEP-02, U4 SW_DP3T, U5 R3006SB

Commit message: 2024/09/22
Parts:
- removed J10: RX==RX, Jumper:SolderJumper-2_P1.3mm_Open_TrianglePad1.0x1.5mm
- removed J11: TX==TX, Jumper:SolderJumper-2_P1.3mm_Open_TrianglePad1.0x1.5mm
- removed J8: RX==TX, Jumper:SolderJumper-2_P1.3mm_Bridged_Pad1.0x1.5mm
- removed J9: TX==RX, Jumper:SolderJumper-2_P1.3mm_Bridged_Pad1.0x1.5mm
- added C3: 2.2u, Footprint_nishi:C_0805_2012, B.Cu at (145.4, 90.1)
- added C4: 2.2u, Footprint_nishi:C_0805_2012, B.Cu at (134.4, 86.1)
- added G***: LOGO, watanabe_smy:YAMADAmain_ver2.0_QR, B.Cu at (136.6, 93.4)
- B_C1, D9, F_C1, Q1, R1, R10, R11, R12, R13, R14, R15, R16, R2, R3, R4, R5, R6, R7, R8, R9, U1, U11, U13, U14, U15, U16, U19, U20, U21, U22, U23: moved to B.Cu
- D10: value Relay_LED -> Relay
- D2: value Batt_LED -> Batt
- D3: value BUSY_LED -> BUSY
- D4: value XMIT_LED -> XMIT
- D5: value SLEEP_LED -> SLEEP
- D6: value STATUS_LED -> STATUS
- D7: value Fuse_LED -> Fuse
- D8: value D_IN_LED -> EMC
- J3: value emc-sw_1 -> EMC:PB9
- U10, U7, U8, U9: value ~ -> NJU7386RB1; footprint SOP8:SOP8 -> watanabe_smy:NJU7386; moved to B.Cu
- U12: value SW_DP3T -> reset
- U4: value SW_DP3T -> REG
- moved Q1 232.8 mm to (160.6, 92.6), turned to 90 degrees
- moved R3 228.8 mm to (160.7, 96.2)
- moved R2 227.3 mm to (160.7, 89.0), turned to 180 degrees
- moved J1 214.1 mm to (157.8, 96.1), turned to 90 degrees
- moved IC1 212.1 mm to (145.5, 95.2), turned to 180 degrees
- moved U5 211.7 mm to (152.3, 79.6)
- moved U4 208.0 mm to (154.3, 115.4)
- moved R12 200.2 mm to (122.2, 116.6)
- moved J5 197.7 mm to (139.9, 113.2), turned to 180 degrees
- moved R13 196.3 mm to (122.2, 115.1)
- moved J4 196.3 mm to (132.4, 113.2), turned to 180 degrees
- moved D11 196.1 mm to (122.0, 116.6), turned to 180 degrees
- moved R14 192.6 mm to (122.2, 113.6)
- moved D12 192.2 mm to (122.0, 115.1), turned to 180 degrees
- moved U8 190.4 mm to (137.8, 113.2), turned to -90 degrees
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Connections:
- U10 pad 1: motor4_A -> M4RIN
- U10 pad 2: Relay_out -> M4FIN
- U10 pad 3: Relay_out -> unconnected-(U10-NC-Pad3)
- U10 pad 4: M4FIN -> motor4_A
- U10 pad 5: M4RIN -> GND
- U10 pad 6: Relay_out -> motor4_B
- U10 pad 7: motor4_B -> unconnected-(U10-NC-Pad7)
- U10 pad 8: GND -> Relay_out
- U18 pad 29: M4RIN -> unconnected-(U18-I2C2_SCL/I2S2_CK/SAI1_SCK_A/SPI2_SCK/TIM2_CH3/USART3_TX/USB_OTG_HS_ULPI_D3/PB10-Pad29)
- U18 pad 31: GND -> Net-(C3-Pad1)
- U18 pad 41: M1RIN -> unconnected-(U18-I2C3_SCL/RCC_MCO_1/TIM1_CH1/USART1_CK/USB_OTG_FS_SOF/PA8-Pad41)
- U18 pad 42: Net-(J11-Pin_2) -> im920sl_RxD
- U18 pad 43: Net-(J10-Pin_2) -> im920sl_TxD
- U18 pad 47: GND -> Net-(C4-Pad1)
- U18 pad 50: unconnected-(U18-ADC1_EXTI15/ADC2_EXTI15/ADC3_EXTI15/CEC/I2S1_WS/I2S3_WS/SPI1_NSS/SPI3_NSS/SYS_JTDI/TIM2_CH1/TIM2_ETR/UART4_RTS/PA15-Pad50) -> M1RIN
- U18 pad 51: unconnected-(U18-PC10/DCMI_D8/I2S3_CK/QUADSPI_BK1_IO1/SDIO_D2/SPI3_SCK/UART4_TX/USART3_TX-Pad51) -> M1FIN
- U18 pad 52: unconnected-(U18-PC11/ADC1_EXTI11/ADC2_EXTI11/ADC3_EXTI11/DCMI_D4/QUADSPI_BK2_NCS/SDIO_D3/SPI3_MISO/UART4_RX/USART3_RX-Pad52) -> M2RIN
- U18 pad 53: unconnected-(U18-PC12/DCMI_D9/I2C2_SDA/I2S3_SD/SDIO_CK/SPI3_MOSI/UART5_TX/USART3_CK-Pad53) -> M2FIN
- U18 pad 55: unconnected-(U18-I2C2_SDA/I2S1_CK/I2S3_CK/SPI1_SCK/SPI3_SCK/SYS_JTDO-SWO/TIM2_CH2/PB3-Pad55) -> M4RIN
- U18 pad 56: M1FIN -> M4FIN
- U18 pad 57: M2RIN -> M3RIN
- U18 pad 58: M2FIN -> M3FIN
- U18 pad 59: M3RIN -> unconnected-(U18-DCMI_VSYNC/I2C1_SDA/SPDIFRX_IN0/TIM4_CH2/USART1_RX/PB7-Pad59)
- U18 pad 61: M3FIN -> unconnected-(U18-CAN1_RX/DCMI_D6/I2C1_SCL/SDIO_D4/TIM10_CH1/TIM2_CH1/TIM2_ETR/TIM4_CH3/PB8-Pad61)
- U18 pad 62: M4FIN -> EMC_IN
- U18 pad 9: EMC_IN -> unconnected-(U18-PC1/ADC1_IN11/ADC2_IN11/ADC3_IN11/I2S2_SD/I2S3_SD/SAI1_SD_A/SPI2_MOSI/SPI3_MOSI-Pad9)
- U5 pad 2: +5V -> BAT
- U6 pad 4: unconnected-(U6-Pad4) -> Relay_out
- U7 pad 1: motor1_A -> M1RIN
- U7 pad 2: Relay_out -> M1FIN
- U7 pad 3: Relay_out -> unconnected-(U7-NC-Pad3)
- U7 pad 4: M1FIN -> motor1_A
- U7 pad 5: M1RIN -> GND
- U7 pad 6: Relay_out -> motor1_B
- U7 pad 7: motor1_B -> unconnected-(U7-NC-Pad7)
- U7 pad 8: GND -> Relay_out
- U8 pad 1: motor2_A -> M2RIN
- U8 pad 2: Relay_out -> M2FIN
- U8 pad 3: Relay_out -> unconnected-(U8-NC-Pad3)
- U8 pad 4: M2FIN -> motor2_A
- U8 pad 5: M2RIN -> GND
- U8 pad 6: Relay_out -> motor2_B
- U8 pad 7: motor2_B -> unconnected-(U8-NC-Pad7)
- U8 pad 8: GND -> Relay_out
- U9 pad 1: motor3_A -> M3RIN
- U9 pad 2: Relay_out -> M3FIN
- U9 pad 3: Relay_out -> unconnected-(U9-NC-Pad3)
- U9 pad 4: M3FIN -> motor3_A
- U9 pad 5: M3RIN -> GND
- U9 pad 6: Relay_out -> motor3_B
- U9 pad 7: motor3_B -> unconnected-(U9-NC-Pad7)
- U9 pad 8: GND -> Relay_out
Routing:
- net +3.3V: track 0.00 -> 147.4 mm, vias 0 -> 9
- net BAT: track 0.00 -> 103.3 mm, vias 0 -> 5
- net Relay_out: track 0.00 -> 78.1 mm, vias 0 -> 6
- net RST: track 0.00 -> 60.5 mm, vias 0 -> 2
- net im920sl_BUSY: track 0.00 -> 57.8 mm, vias 0 -> 3
- net M4FIN: track 0.00 -> 48.7 mm, vias 0 -> 3
- net M2FIN: track 0.00 -> 48.5 mm, vias 0 -> 3
- net SWDIO: track 0.00 -> 46.6 mm
- net im920sl_D-: track 0.00 -> 45.5 mm, vias 0 -> 2
- net im920sl_TxD: track 0.00 -> 44.3 mm, vias 0 -> 2
- net im920sl_zettairesetsaseruMAN: track 0.00 -> 44.3 mm, vias 0 -> 1
- net im920sl_D+: track 0.00 -> 42.2 mm, vias 0 -> 2
- net Net-(U2-IO3/XMIT): track 0.00 -> 42.2 mm, vias 0 -> 1
- net PC_6_Serial6TX: track 0.00 -> 41.9 mm
- net M1FIN: track 0.00 -> 41.9 mm, vias 0 -> 3
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Other:
- board text added: "+3.3V"
- board text added: "+5V"
- board text added: "F446Re"
- board text added: "G +5v SBUS"
- board text added: "M1A:PC10/B:PA15 M2A:PC12/B:PC11"
- board text added: "M3A:PB6/B:PB5 M4A:PB4/B:PB3"
- board text added: "RxD:PA9 TxD:PA10 BUSY:PB1 RESET:PB2"
- board text added: "September.06. 2024 @nnct_robo robo2'_main_board.ver2.0"
- board text added: "TX:PC6/INI:PC8 RX:PC7/RST:PC9"
- board text added: "UART4_RX:PA1"
- board text added: "kottigaue"
- board text removed: "July.05. 2024 @nnct_robo robo2'_main_board.ver1.5"
