File: YAMADAmain_ver2.0/YAMADAmain_ver2.0.kicad_sch (KiCad schematic)
At the start: 53 parts, among them IC1 BD7LS04G-CTL, J1 im920sl_USB, J2 BATT, J3 emc-sw_1, J4 motor1, J5 motor2, J6 motor3, J7 motor4, Q1 2SC3265-Y, U1 NJM2845DL1-33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

Commit message: 2024/09/22
Parts:
- removed U10, U7, U8, U9: ~, SOP8:SOP8, symbol watanabe_sym:BD6211F
- added U10, U7, U8, U9: NJU7386RB1, watanabe_smy:NJU7386, symbol watanabe_sym:NJU7386RB1
Connections:
- net +5V is gone; now on net BAT: U5.2 (5V)
- net GND: now also U10.5 (GND), U7.5 (GND), U8.5 (GND), U9.5 (GND)
- net M1FIN: now also U7.2 (INA)
- net M1RIN: now also U7.1 (INB)
- net M2FIN: now also U8.2 (INA)
- net M2RIN: now also U8.1 (INB)
- net M3FIN: now also U9.2 (INA)
- net M3RIN: now also U9.1 (INB)
- net M4FIN: now also U10.2 (INA)
- net M4RIN: now also U10.1 (INB)
- net Relay_out: now also U6.4, U10.8 (VDD), U7.8 (VDD), U8.8 (VDD), U9.8 (VDD)
- net motor1_A: now also U7.4 (OUTA)
- net motor1_B: now also U7.6 (OUTB)
- net motor2_A: now also U8.4 (OUTA)
- net motor2_B: now also U8.6 (OUTB)
- net motor3_A: now also U9.4 (OUTA)
- net motor3_B: now also U9.6 (OUTB)
- net motor4_A: now also U10.4 (OUTA)
- net motor4_B: now also U10.6 (OUTB)
